Commit message: wheel作成

File: mabot_description/robots/mabot.urdf.xacro (robot description, xacro)
@@ -2,7 +2,16 @@
 <robot name="mabot" xmlns:xacro="http://ros.org/wiki/xacro">
   <xacro:include filename="$(find mabot_description)/urdf/body/body.urdf.xacro"/>
+  <xacro:include filename="$(find mabot_description)/urdf/wheel/wheel.urdf.xacro"/>
   <link name="base_footprint"/>
   <xacro:base parent="base_footprint">
     <origin xyz="0 0 0"/>
   </xacro:base>
+	<xacro:wheel prefix="right" parent="base_link">
+		<origin xyz="0.1 -0.17 0.0" rpy="1.57 0 0" />
+		<axis xyz="0 0 -1" />
+	</xacro:wheel>
+	<xacro:wheel prefix="left" parent="base_link">
+		<origin xyz="0.1 0.17 0.0" rpy="-1.57 0 0" />
+    <axis xyz="0 0 1" />
+  </xacro:wheel>
 </robot>

Commit message: caster作成

File: mabot_description/robots/mabot.urdf.xacro (robot description, xacro)
@@ -3,15 +3,19 @@
   <xacro:include filename="$(find mabot_description)/urdf/body/body.urdf.xacro"/>
   <xacro:include filename="$(find mabot_description)/urdf/wheel/wheel.urdf.xacro"/>
+  <xacro:include filename="$(find mabot_description)/urdf/caster/caster.urdf.xacro"/>
   <link name="base_footprint"/>
   <xacro:base parent="base_footprint">
     <origin xyz="0 0 0"/>
   </xacro:base>
-	<xacro:wheel prefix="right" parent="base_link">
-		<origin xyz="0.1 -0.17 0.0" rpy="1.57 0 0" />
-		<axis xyz="0 0 -1" />
-	</xacro:wheel>
-	<xacro:wheel prefix="left" parent="base_link">
-		<origin xyz="0.1 0.17 0.0" rpy="-1.57 0 0" />
+  <xacro:wheel prefix="right" parent="base_link">
+    <origin xyz="0.1 -0.17 0.0" rpy="1.57 0 0" />
+    <axis xyz="0 0 -1" />
+  </xacro:wheel>
+  <xacro:wheel prefix="left" parent="base_link">
+    <origin xyz="0.1 0.17 0.0" rpy="-1.57 0 0" />
     <axis xyz="0 0 1" />
   </xacro:wheel>
+  <xacro:caster parent="base_link">
+    <origin xyz="-0.15 0 -0.05"/>
+  </xacro:caster>
 </robot>

Commit message: transmission, gazebo pluginの記述

File: mabot_description/robots/mabot.urdf.xacro (robot description, xacro)
@@ -19,3 +19,16 @@
     <origin xyz="-0.15 0 -0.05"/>
   </xacro:caster>
+  <!-- ===========  Transmission ============ -->
+  <xacro:wheel_trans prefix="right" interface="hardware_interface/VelocityJointInterface" />
+  <xacro:wheel_trans prefix="right" interface="hardware_interface/VelocityJointInterface" />
+  <!-- =============== Gazebo =============== -->
+  <gazebo>
+    <plugin name="gazebo_ros_control" filename="libgazebo_ros_control.so">
+      <robotNamespace>mabot</robotNamespace>
+    </plugin>
+  </gazebo>
+  <xacro:base_gazebo/>
+  <xacro:wheel_gazebo prefix="right" />
+  <xacro:wheel_gazebo prefix="left" />
+  <xacro:caster_gazebo/>
 </robot>

File: mabot_description/urdf/body/body.urdf.xacro (robot description, xacro)
@@ -1,4 +1,5 @@
 <?xml version="1.0"?>
 <robot xmlns:xacro="http://ros.org/wiki/xacro">
+  <xacro:include filename="$(find mabot_description)/urdf/body/body.gazebo.xacro" />
   <xacro:property name="M_PI" value="3.1415926535897931" />
   <xacro:property name="velocity_scale_factor" value="1.0"/>

File: mabot_description/urdf/caster/caster.urdf.xacro (robot description, xacro)
@@ -1,4 +1,5 @@
 <?xml version="1.0"?>
 <robot xmlns:xacro="http://ros.org/wiki/xacro">
+  <xacro:include filename="$(find mabot_description)/urdf/body/body.gazebo.xacro" />
   <xacro:macro name="caster" params="parent *joint_origin">
     <joint name="$caster_joint" type="fixed">

File: mabot_description/urdf/wheel/wheel.urdf.xacro (robot description, xacro)
@@ -1,4 +1,6 @@
 <?xml version="1.0"?>
 <robot xmlns:xacro="http://ros.org/wiki/xacro">
+  <xacro:include filename="$(find mabot_description)/urdf/wheel/wheel.gazebo.xacro" />
+  <xacro:include filename="$(find mabot_description)/urdf/wheel/wheel.transmission.xacro" />
   <xacro:macro name="wheel" params="prefix parent *joint_origin *joint_axis">
     <joint name="${prefix}_wheel_joint" type="continuous">
@@ -19,9 +21,9 @@
         </geometry>
       </collision>
-        <inertial>
-          <origin xyz="0.0 0.0 0.0" />
-          <mass value="0.500"/>
-          <inertia ixx="0.0013541667" ixy="0" ixz="0" iyy="0.0013541667" iyz="0" izz="0.0025"/>
-        </inertial>
+      <inertial>
+        <origin xyz="0.0 0.0 0.0" />
+        <mass value="0.500"/>
+        <inertia ixx="0.0013541667" ixy="0" ixz="0" iyy="0.0013541667" iyz="0" izz="0.0025"/>
+      </inertial>
     </link>
   </xacro:macro>

Commit message: fix wheel_separation

File: mabot_description/robots/mabot.urdf.xacro (robot description, xacro)
@@ -9,9 +9,9 @@
   </xacro:base>
   <xacro:wheel prefix="right" parent="base_link">
-    <origin xyz="0.1 -0.17 0.0" rpy="1.57 0 0" />
+    <origin xyz="0.1 -0.13 0.0" rpy="1.57 0 0" />
     <axis xyz="0 0 -1" />
   </xacro:wheel>
   <xacro:wheel prefix="left" parent="base_link">
-    <origin xyz="0.1 0.17 0.0" rpy="-1.57 0 0" />
+    <origin xyz="0.1 0.13 0.0" rpy="-1.57 0 0" />
     <axis xyz="0 0 1" />
   </xacro:wheel>

Commit message: Add material

File: mabot_description/robots/mabot.urdf.xacro (robot description, xacro)
@@ -25,5 +25,5 @@
   <gazebo>
     <plugin name="gazebo_ros_control" filename="libgazebo_ros_control.so">
-      <robotNamespace>mabot</robotNamespace>
+      <robotNamespace>/mabot</robotNamespace>
     </plugin>
   </gazebo>

File: mabot_description/urdf/body/body.urdf.xacro (robot description, xacro)
@@ -15,4 +15,7 @@
           <box size="0.400 0.200 0.100"/>
         </geometry>
+        <material name="gray">
+          <color rgba="1 1 1 1"/>
+        </material>
       </visual>
       <collision>

File: mabot_description/urdf/caster/caster.urdf.xacro (robot description, xacro)
@@ -13,4 +13,7 @@
           <sphere radius="0.05"/>
         </geometry>
+        <material name="cyan">
+          <color rgba="0 1 1 1"/>
+        </material>
       </visual>
       <collision>

File: mabot_description/urdf/wheel/wheel.urdf.xacro (robot description, xacro)
@@ -15,4 +15,7 @@
           <cylinder radius="0.1" length="0.05"/>
         </geometry>
+        <material name="yellow">
+          <color rgba="1 1 0 1"/>
+        </material>
       </visual>
       <collision>

Commit message: Remove: mabot_lrf

File: mabot_description/robots/mabot.urdf.xacro (robot description, xacro)
@@ -4,4 +4,5 @@
   <xacro:include filename="$(find mabot_description)/urdf/wheel/wheel.urdf.xacro"/>
   <xacro:include filename="$(find mabot_description)/urdf/caster/caster.urdf.xacro"/>
+  <xacro:include filename="$(find mabot_description)/urdf/sensors/lrf.urdf.xacro"/>
   <link name="base_footprint"/>
   <xacro:base parent="base_footprint">
@@ -16,4 +17,7 @@
     <axis xyz="0 0 1" />
   </xacro:wheel>
+  <xacro:lrf_sensor prefix="top" parent="base_link">
+    <origin xyz="0 0 0.2" rpy="0 0 0" />
+  </xacro:lrf_sensor>
   <xacro:caster parent="base_link">
     <origin xyz="-0.15 0 -0.05"/>
@@ -32,3 +36,4 @@
   <xacro:wheel_gazebo prefix="left" />
   <xacro:caster_gazebo/>
+  <xacro:lrf_gazebo prefix="top" rad_range="${radians(180)}" min_range="0.1" max_range="5.0"/>
 </robot>
